File: backlight.kicad_pcb (KiCad board)
At the start: 2 copper layers, 150 x 90 mm, 52 parts, among them J1 Screw_Terminal_01x03, U1 SY7203

Commit message: upd
Parts:
- moved D41 26.2 mm to (58.3, 60.2)
- moved L1 23.8 mm to (64.5, 56.9), turned to 0 degrees
- moved C1 23.5 mm to (61.1, 62.6)
- moved C2 22.7 mm to (55.5, 63.2), turned to -90 degrees
- moved R6 19.6 mm to (67.4, 63.8), turned to -90 degrees
- moved U1 17.4 mm to (64.3, 62.4), turned to 180 degrees
- moved J1 17.1 mm to (49.9, 62.0)
- moved R2 1.30 mm to (190.1, 75.2)
- moved R3 1.30 mm to (190.1, 96.2)
- moved R4 1.30 mm to (190.1, 116.2)
- moved R5 1.30 mm to (190.1, 123.0)
Routing:
- net /LED+: track 17.1 -> 98.1 mm
- net /LED-: track 138.8 -> 204.8 mm
- net Net-(D30-K): track 0.00 -> 19.0 mm
- net Net-(D4-K): track 0.00 -> 18.7 mm
- net Net-(D33-K): track 0.00 -> 17.7 mm
- net Net-(D25-K): track 0.00 -> 17.7 mm
- net Net-(D17-K): track 0.00 -> 17.7 mm
- net Net-(D10-A): track 0.00 -> 17.7 mm
- net Net-(D1-K): track 0.00 -> 17.7 mm
- net Net-(D7-K): track 0.00 -> 17.7 mm
- net Net-(D6-K): track 0.00 -> 17.7 mm
- net Net-(D5-K): track 0.00 -> 17.7 mm
- net Net-(D39-K): track 0.00 -> 17.7 mm
- net Net-(D38-K): track 0.00 -> 17.7 mm
- net Net-(D37-K): track 0.00 -> 17.7 mm
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
Commit message: test (#1)
Merge routing
Parts:
- moved R5 1.05 mm to (191.1, 123.1)
- moved R1 0.98 mm to (190.9, 55.8)
- moved R2 0.88 mm to (190.9, 75.1)
- moved R3 0.87 mm to (190.9, 96.2)
- moved R4 0.72 mm to (190.8, 116.2)
Routing:
- net /LED-: track 204.8 -> 200.6 mm
- net Net-(D30-K): track 19.0 -> 17.1 mm
- net Net-(D8-K): track 5.46 -> 4.19 mm
- net Net-(D24-K): track 5.62 -> 4.43 mm
- net Net-(D16-K): track 4.62 -> 3.43 mm
- net Net-(D4-K): track 18.7 -> 17.6 mm
- net Net-(D36-K): track 17.7 -> 16.8 mm
- net Net-(D11-K): track 17.7 -> 16.8 mm
- net Net-(D28-K): track 17.7 -> 16.8 mm
- net Net-(D20-K): track 17.7 -> 16.9 mm
- net Net-(D38-K): track 17.7 -> 16.9 mm
- net Net-(D17-K): track 17.7 -> 16.9 mm
- net Net-(D25-K): track 17.7 -> 16.9 mm
- net Net-(D37-K): track 17.7 -> 16.9 mm
- net Net-(D15-K): track 17.7 -> 16.9 mm
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- added copper zone on F.Cu, net /LED+
- added copper zone on F.Cu, net GND
- added copper zone on F.Cu, net VPP
