File: backlight.kicad_sch (KiCad schematic)
At the start: 52 parts, among them J1 Screw_Terminal_01x03, U1 SY7203

Commit message: Reroute board
Parts:
- removed D41: D_Schottky, Diode_SMD:D_SMA, symbol Device:D_Schottky
- removed J1: Screw_Terminal_01x03, Connector_PinHeader_2.54mm:PinHeader_1x03_P2.54mm_Vertical_SMD_Pin1Left, symbol Connector:Screw_Terminal_01x03
- added D41: SS24, Diode_SMD:D_SMA, symbol Diode:SS24
- added J1: Conn_01x03_MountingPin, rainwalker:XH254-0,5-3-2,5-V-SMD_1x03-1MP_P2.50mm_Vertical, symbol Connector_Generic_MountingPin:Conn_01x03_MountingPin
- added R7: 10k, Resistor_SMD:R_0805_2012Metric, symbol Device:R
- C1: value C -> 4.7uF 35V
- C2: value C -> 2.2uF 35V
- R6: value R -> 2R
- U1: footprint Package_DFN_QFN:DFN-10-1EP_3x3mm_P0.5mm_EP1.75x2.7mm -> rainwalker:SY7203DBC-DFN-10-1EP_3x3mm_P0.5mm_EP1.75x2.7mm
Connections:
- net EN_PWM: now also J1.2 (Pin_2), R7.1
- net GND: now also J1.1 (Pin_1), J1.MP (MountPin), R7.2
- net LED+: now also D41.1 (K)
- net VPP: now also J1.3 (Pin_3)
- net at L1.2, U1.4 (LX), U1.5 (LX): now also D41.2 (A)
